Commit message: feat: Completed Phase 1 - Upgraded simulation to Gazebo

File: description/boat.urdf (robot description, URDF)
Before this commit: robot boat, 1 links, 0 joints
Links:
- added link camera_link; visual box size=0.05 0.05 0.05
- link base_link: mass None -> 10.0; geometry collision box size=1.0 0.5 0.3; visual box size=1.0 0.5 0.3
Joints:
- added joint camera_joint: type fixed, parent base_link, child camera_link, origin xyz=0.5 0 0.2 rpy=0 0 0
